Commit message: mcl/kalman update

File: src/puzzlebot_description/models/puzzlebot/puzzlebot.urdf (robot description, URDF)
Before this commit: robot Puzzlebot_Jetson_Lidar_Ed., 7 links, 6 joints
Links:
- removed link base_footprint
- removed link camera_base_link
- removed link caster_holder_link
- removed link lidar_base_link
- removed link wheel_left_link
- removed link wheel_right_link
- added link camera_link, mass 0.01; visual box size=0.02 0.02 0.02
- added link chassis, mass 0.8; collision mesh filename=package://puzzlebot_description/models/puzzlebot/meshes/cha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; visual mesh filename=package://puzzlebot_description/models/puzzlebot/meshes/cha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
- added link left_wheel, mass 0.05; collision mesh filename=package://puzzlebot_description/models/puzzlebot/meshes/whe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; visual mesh filename=package://puzzlebot_description/models/puzzlebot/meshes/whe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
- added link right_wheel, mass 0.05; collision mesh filename=package://puzzlebot_description/models/puzzlebot/meshes/whe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; visual mesh filename=package://puzzlebot_description/models/puzzlebot/meshes/whe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
- link base_link: mass None -> 0.0001; geometry 
Joints:
- removed joint base_link_joint
- removed joint camera_base_joint
- removed joint caster_holder_joint
- removed joint lidar_base_joint
- removed joint wheel_left_joint
- removed joint wheel_right_joint
- added joint camera_joint: type fixed, parent chassis, child camera_link, origin xyz=0.1 0 0.08 rpy=0 0 0
- added joint chassis_joint: type fixed, parent base_link, child chassis, origin xyz=0 0 0 rpy=0 0 0
- added joint left_wheel_joint: type revolute, parent chassis, child left_wheel, origin xyz=0.05 0.09 0.05 rpy=0 0 0, axis 0 1 0, limit lower=-1.79769e+308 upper=1.79769e+308 effort=1 velocity=6
- added joint right_wheel_joint: type revolute, parent chassis, child right_wheel, origin xyz=0.05 -0.09 0.05 rpy=0 0 0, axis 0 1 0, limit lower=-1.79769e+308 upper=1.79769e+308 effort=1 velocity=6
