Commit message: gz update

File: src/puzzlebot_description/models/puzzlebot/model.urdf (robot description, URDF)
Before this commit: robot puzzlebot, 5 links, 4 joints
Links:
- added link caster, mass 0.01; collision sphere radius=0.006; visual sphere radius=0.006
- added link lidar_link, mass 0.1; collision mesh filename=package://puzzlebot_description/models/puzzlebot/meshes/LiD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 scale=0.001 0.001 0.001; visual mesh filename=package://puzzlebot_description/models/puzzlebot/meshes/LiD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 scale=0.001 0.001 0.001
Joints:
- removed joint wheel_left_joint
- removed joint wheel_right_joint
- added joint caster_wheel: type fixed, parent chassis, child caster, origin xyz=-0.095 0.0 0.006 rpy=0 0 0
- added joint left_wheel_joint: type revolute, parent chassis, child left_wheel, origin xyz=0.052 0.095 -0.0025 rpy=0 0 0, axis 0 1 0, limit lower=-1.79769e+308 upper=1.79769e+308 effort=1 velocity=6
- added joint lidar_joint: type fixed, parent chassis, child lidar_link, origin xyz=0.045 0 0.138 rpy=0 0 0
- added joint right_wheel_joint: type revolute, parent chassis, child right_wheel, origin xyz=0.052 -0.095 -0.0025 rpy=0 0 0, axis 0 1 0, limit lower=-1.79769e+308 upper=1.79769e+308 effort=1 velocity=6

Commit message: rviz fix

File: src/puzzlebot_description/models/puzzlebot/model.urdf (robot description, URDF)
Before this commit: robot puzzlebot, 7 links, 6 joints
Joints:
- joint left_wheel_joint: limit lower=-1.79769e+308 upper=1.79769e+308 effort=1 velocity=6 -> (none); origin xyz=0.052 0.095 -0.0025 rpy=0 0 0 -> xyz=0.05 0.09 0.05 rpy=0 0 0; type revolute -> continuous
- joint right_wheel_joint: limit lower=-1.79769e+308 upper=1.79769e+308 effort=1 velocity=6 -> (none); origin xyz=0.052 -0.095 -0.0025 rpy=0 0 0 -> xyz=0.05 -0.09 0.05 rpy=0 0 0; type revolute -> continuous

Commit message: cartographer_adaptation fix

File: src/puzzlebot_description/models/puzzlebot/model.urdf (robot description, URDF)
Before this commit: robot puzzlebot, 7 links, 6 joints
Joints:
- joint lidar_joint: origin xyz=0.045 0 0.138 rpy=0 0 0 -> xyz=0.045 0 0.138 rpy=3.141592 0 -3.141592
